File: water_meter.kicad_sch (KiCad schematic)
At the start: 50 parts, among them J1 2464, J2 Conn_01x02_Male, J3 Conn_01x06_Male, J4 USB_Micro-10118193-0001LF, J5 Conn_01x02_Male, J8 Conn_01x02_Male, U1 RT9080-33GJ5, U2 ESP32-S3-WROOM-1, U3 ALT025-10E, U4 SLG46826G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

Commit message: V2
Parts:
- removed CLK1, INT1, PIN4, PIN5, SCL1, SDA1, VBAT1: TestPoint, TestPoint:TestPoint_Pad_D2.0mm, symbol Connector:TestPoint
- removed D1: WS2812B, LED_SMD:LED_WS2812B_PLCC4_5.0x5.0mm_P3.2mm, symbol LED:WS2812B
- removed J2: Conn_01x02_Male, Connector_PinSocket_2.54mm:PinSocket_1x02_P2.54mm_Vertical, symbol Connector:Conn_01x02_Male
- removed Y1: 32.768kHz (ESR < 70 kΩ), Crystal:Crystal_SMD_G8-2Pin_3.2x1.5mm_HandSoldering, symbol water_meter-rescue:Crystal-Device
- removed Y2: Crystal, Crystal:Crystal_C38-LF_D3.0mm_L8.0mm_Vertical, symbol Device:Crystal
- added C16: 0.1uF, Capacitor_SMD:C_0805_2012Metric, symbol water_meter-rescue:C_Small-Device
- added Q1, Q2: BSS84, Package_TO_SOT_SMD:SOT-23, symbol Transistor_FET:BSS84
- added R10, R8: 100k, Resistor_SMD:R_0805_2012Metric, symbol water_meter-rescue:R_Small-Device
- added R11: 2k, Resistor_SMD:R_0805_2012Metric, symbol water_meter-rescue:R_Small-Device
- added R12: 1k, Resistor_SMD:R_0805_2012Metric, symbol water_meter-rescue:R_Small-Device
- added R13: 500R, Resistor_SMD:R_0805_2012Metric, symbol water_meter-rescue:R_Small-Device
- added U6: IN-PI22TAT5R5G5B, Nabil:INPI22TAT5R5G5B, symbol Nabil:IN-PI22TAT5R5G5B
- added U7: 10413_lens, Nabil:10414_Lens, symbol Nabil:10413_lens
- added U8: MB85RC64TA, Package_SO:SOIC-8_3.9x4.9mm_P1.27mm, symbol Memory_NVRAM:FM24C64C
- added Y1, Y2: ABS07-32.768KHZ-T, Nabil:XTAL_ABS07-32.768KHZ-T, symbol Nabil:ABS07-32.768KHZ-T
- C1, C10, C11, C12, C13, C14, C15, C2, C3, C4, C6, C7, C8, C9: footprint Capacitor_SMD:C_0805_2012Metric_Pad1.18x1.45mm_HandSolder -> Capacitor_SMD:C_0805_2012Metric
- C5: value 10uF/25V(20%) -> 10uF; footprint Capacitor_SMD:C_0805_2012Metric_Pad1.18x1.45mm_HandSolder -> Capacitor_SMD:C_0805_2012Metric
- D2: footprint LED_SMD:LED_0805_2012Metric_Pad1.15x1.40mm_HandSolder -> LED_SMD:LED_0805_2012Metric
- F1: footprint Fuse:Fuse_1206_3216Metric_Pad1.42x1.75mm_HandSolder -> Fuse:Fuse_1206_3216Metric; Mouser Part Number (none) -> 652-MF-NSMF110-2
- H1, H2, H3, H4: footprint MountingHole:MountingHole_2.5mm -> MountingHole:MountingHole_2.5mm_Pad
- J4: Mouser Part Number (none) -> 649-10118193-0001LF
- R1: value 10k(1%) -> 10k; footprint Resistor_SMD:R_0805_2012Metric_Pad1.20x1.40mm_HandSolder -> Resistor_SMD:R_0805_2012Metric
- R2, R3, R4, R5, R7, R9: footprint Resistor_SMD:R_0805_2012Metric_Pad1.20x1.40mm_HandSolder -> Resistor_SMD:R_0805_2012Metric
- R6: value 5.1K -> 4.7k; footprint Resistor_SMD:R_0805_2012Metric_Pad1.20x1.40mm_HandSolder -> Resistor_SMD:R_0805_2012Metric
- U1: Digikey Part Number (none) -> 1028-1509-1-ND
- U2: footprint Espressif:ESP32-S3-WROOM-1 -> Espressif:ESP32-S3-WROOM-1U; Mouser Part Number (none) -> 356-ESP32S3WROM1UN16
- U4: Mouser Part Number (none) -> 724-SLG46826G
- U5: Mouser Part Number (none) -> 771-PCF8563TS/5118
Connections:
- net +3V3: now also Q1.2 (S), Q2.2 (S), R12.2, R8.2, U8.8 (VDD); no longer J5.2 (Pin_2), U3.6 (VCC), U4.20 (VDD)
- net GND: now also C16.1, R10.1, U6.2 (VSS), U8.4 (VSS)
- net LED_PIN0: now also R11.2; no longer C15.1
- net M_CLK: now also R8.1
- net SCL: now also U8.6 (SCL)
- net SDA: now also U8.5 (SDA)
- net SLG_INT2: now also U4.8 (IO8); no longer U4.9 (IO7)
- net VBATT: now also J1.1 (+)
- net MAG_PWR: now reaches U4.5 (IO10)
- net MAG_PWR: now also U3.6 (VCC)
- net at C2.2, R3.2: now also Y1.1
- net at C7.2, U5.1 (OSCI): now also Y2.2
- net at C1.2, R2.2: now also Y1.2
- net at C13.2, U5.2 (OSCO): now also Y2.1
- net RTC_INT: now reaches U5.3 (~{INT})
- net RTC_INT: now also U2.6 (GPIO6/TOUCH6/ADC1_CH5)
- net LED_PWR: now reaches U2.39 (GPIO1/TOUCH1/ADC1_CH0)
- net LED_PWR: now also R13.1
- net SLG_PWR_GPIO: now reaches U2.7 (GPIO7/TOUCH7/ADC1_CH6)
- net SLG_PWR_GPIO: now also Q1.1 (G), R10.2
- new net: Q2.1 (G), R12.1, R13.2
- new net: C15.1, Q2.3 (D), U6.4 (VDD)
- new net: R11.1, U6.3 (DIN)
- new net SLG_PWR: C16.2, J5.2 (Pin_2), Q1.3 (D), U4.20 (VDD)
- no-connect marks 35 -> 38
Other:
- moved on the sheet: C11, C12, C13, C14, C15, C2, C5, C7, C8, D2, F1, J4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

Commit message: V3
Parts:
- removed C11, C12: 100pF, Capacitor_SMD:C_0805_2012Metric, symbol water_meter-rescue:C_Small-Device
- removed C16: 0.1uF, Capacitor_SMD:C_0805_2012Metric, symbol water_meter-rescue:C_Small-Device
- removed H1, H2, H3, H4: MountingHole_Pad, MountingHole:MountingHole_2.5mm_Pad, symbol water_meter-rescue:MountingHole_Pad-Mechanical
- removed J5: Conn_01x02_Male, Jumper:SolderJumper-2_P1.3mm_Bridged_Pad1.0x1.5mm, symbol Connector:Conn_01x02_Male
- removed J8: Conn_01x02_Male, Connector_PinSocket_2.54mm:PinSocket_1x02_P2.54mm_Vertical, symbol Connector:Conn_01x02_Male
- removed Q1: BSS84, Package_TO_SOT_SMD:SOT-23, symbol Transistor_FET:BSS84
- removed U3: ALT025-10E, Nabil:SON65P250X250X80-7N, symbol Nabil:ALT025-10E
- removed U4: SLG46826G, Nabil:SOP65P640X120-20N, symbol Nabil:SLG46826G
- removed U7: 10413_lens, Nabil:10414_Lens, symbol Nabil:10413_lens
- added C17, C19: 0.1uF, Capacitor_SMD:C_0805_2012Metric, symbol water_meter-rescue:C_Small-Device
- added H1, H2, H3, H4: MountingHole, MountingHole:MountingHole_6mm, symbol Mechanical:MountingHole
- added J6: Conn_01x08_Female, Connector_JST:JST_SH_SM08B-SRSS-TB_1x08-1MP_P1.00mm_Horizontal, symbol Connector:Conn_01x08_Female
- added J7: Conn_01x04_Female, Connector_JST:JST_SH_SM04B-SRSS-TB_1x04-1MP_P1.00mm_Horizontal, symbol Connector:Conn_01x04_Female
- added Q3: BSS84, Package_TO_SOT_SMD:SOT-23, symbol Transistor_FET:BSS84
- added R14: 10M, Resistor_SMD:R_0805_2012Metric, symbol water_meter-rescue:R_Small-Device
- added S1: PTS526_SK15_SMTR2_LFS, Nabil:PTS526SK15SMTR2LFS, symbol Nabil:PTS526_SK15_SMTR2_LFS
- R10: value 100k -> 10M
- R12: value 1k -> 10k
Connections:
- net +3V3: now also J6.6 (Pin_6), J7.2 (Pin_2)
- net EN: now also C17.1, S1.1, S1.2
- net GND: now also C17.2, C19.2, J6.8 (Pin_8), J7.4 (Pin_4), Q3.1 (G), R14.2, S1.3, S1.4; no longer R10.1
- net M_CLK: now also J6.7 (Pin_7)
- net SCL: now also J6.5 (Pin_5)
- net SDA: now also J6.4 (Pin_4)
- net SLG_INT1: now also J6.1 (Pin_1)
- net SLG_INT2: now also J6.2 (Pin_2)
- net VBATT: now also R10.1, Q3.2 (S); no longer J1.1 (+)
- net RTC_INT: no longer names the net of U5.3 (~{INT})
- net RTC_INT: no longer U2.6 (GPIO6/TOUCH6/ADC1_CH5)
- net SLG_PWR_GPIO renamed MAG
- net MAG: now also J6.3 (Pin_3), J7.3 (Pin_3); no longer R10.2
- new net: J1.1 (+), Q3.3 (D)
- new net SLG_PIN19: J7.1 (Pin_1)
- new net VBATT_DIV: C19.1, R10.2, R14.1, U2.6 (GPIO6/TOUCH6/ADC1_CH5)
- no-connect marks 38 -> 27
Other:
- added sheet Sensors (sensors.kicad_sch)
- note added: "Strapping pins for ESP32S3: • GPIO0 • GPIO45 • GPIO46 • GPIO3"
- moved on the sheet: C4, C5, C6, F1, J1, J4, R5, R7

Commit message: Prototype V0.4   - New board layout for new enclosure   - Added user button   - Using opamp power down pin to save power
Parts:
- removed J1: 2464, Nabil:2464, symbol Nabil:2464
- removed J4: USB_Micro-10118193-0001LF, Nabil:FCI_10118193-0001LF, symbol Nabil:USB_Micro-10118193-0001LF
- removed J6: Conn_01x08_Female, Connector_JST:JST_SH_SM08B-SRSS-TB_1x08-1MP_P1.00mm_Horizontal, symbol Connector:Conn_01x08_Female
- removed J7: Conn_01x04_Female, Connector_JST:JST_SH_SM04B-SRSS-TB_1x04-1MP_P1.00mm_Horizontal, symbol Connector:Conn_01x04_Female
- removed Q3: BSS84, Package_TO_SOT_SMD:SOT-23, symbol Transistor_FET:BSS84
- added C20: 0.1uF, Capacitor_SMD:C_0805_2012Metric, symbol water_meter-rescue:C_Small-Device
- added J1: Conn_01x02_Female, Nabil:JST_PH_B2B-PH-SM4-TB_1x02-1MP_P2.00mm_Vertical, symbol Connector:Conn_01x02_Female
- added J4: USB_B_Micro, Nabil:USB_Micro-B_Molex-105133-0001, symbol Connector:USB_B_Micro
- added J6: 2465, Nabil:2465, symbol Nabil:2465
- added Q1: BSS84, Package_TO_SOT_SMD:SOT-23, symbol Transistor_FET:BSS84
- added Q3, Q4: MMBT3904, Package_TO_SOT_SMD:SOT-23, symbol Transistor_BJT:MMBT3904
- added R20: 10k, Resistor_SMD:R_0805_2012Metric, symbol water_meter-rescue:R_Small-Device
- added R21, R22: 10K, Resistor_SMD:R_0805_2012Metric_Pad1.20x1.40mm_HandSolder, symbol Device:R_Small
- added S2: PTS526_SK15_SMTR2_LFS, Nabil:PTS526SK15SMTR2LFS, symbol Nabil:PTS526_SK15_SMTR2_LFS
- H1, H2, H3, H4: footprint MountingHole:MountingHole_6mm -> MountingHole:MountingHole_3.2mm_M3
Connections:
- net +3V3: now also R20.1
- net EN: now also Q3.3 (C); no longer J3.6 (Pin_6)
- net GND: now also C20.2, J1.2 (Pin_2), J4.5 (GND), J4.6 (Shield), Q1.1 (G), S2.3, S2.4
- net GPIO0: now also Q4.3 (C); no longer J3.2 (Pin_2)
- net USB_D+: now also J4.3 (D+)
- net USB_D-: now also J4.2 (D-)
- net VBATT: now also Q1.2 (S)
- net at F1.2: now also J4.1 (VBUS)
- net USER_INPUT: now reaches U2.35 (MTMS/GPIO42)
- net USER_INPUT: now also C20.1, R20.2, S2.1, S2.2
- new net: Q3.1 (B), R21.1
- new net: J1.1 (Pin_1), Q1.3 (D)
- new net: Q4.1 (B), R22.1
- new net DTR: J3.6 (Pin_6), Q4.2 (E), R21.2
- new net RTS: J3.2 (Pin_2), Q3.2 (E), R22.2
- no-connect marks 27 -> 26
Other:
- sheet Sensors ports: added none; removed SLG_PIN19, VBATT_DIV
- moved on the sheet: C5, F1, J3, U8
